File: PCB/ESC_v3/ESC_v3.kicad_pcb (KiCad board)
At the start: 4 copper layers, 42 x 83.5 mm, 140 parts, among them IC1 TLV77333PDBVR, J1 Conn_01x02_Pin, J1 Conn_01x04_Pin, J10 Conn_01x01_Pin, J11 Screw_Terminal_01x01, J2 Screw_Terminal_01x01, J3 Conn_01x01_Pin, J4 Conn_01x01_Pin, J5 Conn_01x01_Pin, J6 Conn_01x01_Pin, J7 Conn_01x01_Pin, J8 Conn_01x01_Pin, J9 Conn_01x01_Pin, Q1 NTMFS2D1N08XT1G, Q2 NTMFS2D1N08XT1G, Q3 NTMFS2D1N08XT1G, Q4 NTMFS2D1N08XT1G, Q5 NTMFS2D1N08XT1G, Q6 NTMFS2D1N08XT1G, U1 SN65HVD232, U2 DRV8323SRTAT, U3 STM32G474CETx, Y2 24MHz

Commit message: Layout update
Parts:
- removed G*** (x2): LOGO, LOGO
- removed H3: MountingHole_Pad, MountingHole:MountingHole_3.2mm_M3_ISO14580_Pad
- removed the J1 at (133.4, 116.6)
- removed J11, J2: Screw_Terminal_01x01, TerminalBlock_Wuerth:Wuerth_REDCUBE-THR_WP-THRSH_74651173_THR
- removed L2: 6.8uH, Inductor_SMD:L_0805_2012Metric_Pad1.05x1.20mm_HandSolder
- removed U1: SN65HVD232, Package_SO:SOIC-8_3.9x4.9mm_P1.27mm
- removed U2: DRV8323SRTAT, DRV8323SRTAT:QFN50P600X600X80-41N415X415
- added C49: 1u, Capacitor_SMD:C_0603_1608Metric, F.Cu at (141.8, 91.3)
- added C50: 4u7, Capacitor_SMD:C_0805_2012Metric, B.Cu at (150.0, 43.3)
- added C52: 4u7, Capacitor_SMD:C_0805_2012Metric, B.Cu at (139.5, 43.5)
- added C53: 4u7, Capacitor_SMD:C_0805_2012Metric, B.Cu at (129.0, 43.4)
- added D10: LED, LED_SMD:LED_0805_2012Metric, F.Cu at (127.4, 103.0)
- added D7: LED, LED_SMD:LED_0805_2012Metric, F.Cu at (127.4, 100.6)
- added FB1: FCM1608KF-601T03, Inductor_SMD:L_0603_1608Metric, F.Cu at (145.0, 90.3)
- added IC2: TCAN3414DR, SamacSys_Parts:SOIC127P600X175-8N, B.Cu at (133.2, 96.6)
- added IC3: DRV8323SRTAR, SamacSys_Parts:QFN50P600X600X80-41N-D, F.Cu at (145.4, 66.6)
- added PS1: XT60PW-M, SamacSys_Parts:XT60PWM, F.Cu at (152.7, 99.5)
- added R32: 10, Resistor_SMD:R_0402_1005Metric, F.Cu at (143.2, 89.1)
- added R33: 2k, Resistor_SMD:R_0603_1608Metric, F.Cu at (133.3, 100.6)
- added R49: 2k, Resistor_SMD:R_0603_1608Metric, F.Cu at (133.3, 103.0)
- C15, C18, C4: value 1µF/50V -> 4u7
- C16: footprint Capacitor_SMD:C_0805_2012Metric -> Capacitor_SMD:C_0402_1005Metric
- C17, C27, C29, C30, C31: moved to F.Cu
- C19, C26, C51, R38: moved to B.Cu
- C35, C43: footprint Capacitor_SMD:C_0603_1608Metric -> Capacitor_SMD:C_0402_1005Metric
- C39, C42: value 1u/DNP -> 1u
- C40, C41: footprint Capacitor_SMD:C_0805_2012Metric -> Capacitor_SMD:C_0603_1608Metric
- C46, C47: value 12pF -> 100p; footprint Capacitor_SMD:C_0603_1608Metric -> Capacitor_SMD:C_0402_1005Metric
- C48: value 12pF -> 100p; footprint Capacitor_SMD:C_0805_2012Metric -> Capacitor_SMD:C_0402_1005Metric
- D1: value SMCJ28A -> SMCJ33A-TR; footprint Diode_SMD:D_SMC -> SamacSys_Parts:SMCJ15ATR
- Q1, Q2, Q3, Q4, Q5, Q6: value NTMFS2D1N08XT1G -> NTMFS5C670NLT1G; footprint Package_SO:ONSemi_SO-8FL_488AA -> SamacSys_Parts:NRVTS10100EMFST1G
- R25, R29, R30: value 3m -> 1m; footprint Resistor_SMD:R_2512_6332Metric -> SamacSys_Parts:RESC6432X110N
- R46, R47, R48: value 100 -> 33; footprint Resistor_SMD:R_0603_1608Metric -> Resistor_SMD:R_0402_1005Metric
- moved R48 24.3 mm to (149.5, 84.8)
- moved C27 23.7 mm to (160.5, 86.2)
- moved R46 23.1 mm to (134.5, 86.6), turned to 180 degrees
- moved J8 20.7 mm to (127.3, 92.5), turned to -90 degrees
- moved R47 20.3 mm to (134.5, 85.3), turned to 180 degrees
- moved C29 18.9 mm to (160.5, 64.8)
- moved C51 17.6 mm to (160.1, 67.3)
- moved C26 17.6 mm to (160.1, 84.9)
- moved J7 17.5 mm to (143.0, 97.8)
- moved H4 17.5 mm to (145.2, 110.0)
- moved J10 16.3 mm to (127.3, 95.1), turned to -90 degrees
- moved J4 13.9 mm to (145.6, 103.0)
- moved J5 12.8 mm to (143.0, 103.0)
- moved J6 12.8 mm to (143.0, 100.4)
- moved C17 12.7 mm to (133.2, 96.2), turned to 180 degrees
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Connections:
- C35 pad 2: VREF -> +VDDA
- C39 pad 2: VREF -> +VDDA
- C43 pad 2: VREF -> +VREF
- R25 pad 1: SPA -> GND
- R25 pad 2: GND -> SPA
- R29 pad 1: SPB -> GND
- R29 pad 2: GND -> SPB
- R30 pad 1: SPC -> GND
- R30 pad 2: GND -> SPC
- U3 pad 18: unconnected-(U3-PB2-Pad18) -> DBG_LED
- U3 pad 20: VREF -> +VREF
- U3 pad 21: VREF -> +VDDA
Routing:
- net ADC2_IN17: track 38.3 -> 3.19 mm
- net ADC4_IN4: track 35.8 -> 2.70 mm, vias 2 -> 0
- net SOA: track 9.34 -> 42.4 mm, vias 0 -> 2
- net SOC: track 8.57 -> 40.5 mm
- net ADC1_IN4: track 32.1 -> 3.19 mm
- net SOB: track 8.65 -> 36.6 mm
- net +3V3: track 118.6 -> 97.3 mm, vias 9 -> 11
- net V_BAT: track 82.1 -> 64.1 mm, vias 90 -> 1
- net DBG_LED: track 0.00 -> 17.3 mm, vias 0 -> 2
- net NRST: track 39.2 -> 26.6 mm
- net USART2_TX: track 28.7 -> 16.3 mm
- net VREF: track 9.11 -> 0.00 mm
- net SWCLK: track 34.3 -> 25.6 mm
- net +VDDA: track 0.00 -> 5.53 mm
- net CAN_TX: track 14.5 -> 19.6 mm
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- removed copper zone on In2.Cu, net V_A_PHASE
- removed copper zone on In2.Cu, net V_BAT
- removed copper zone on In2.Cu, net V_B_PHASE
- removed copper zone on In2.Cu, net V_C_PHASE
Other:
- board text added: "ESC v1 03/26"
- board text removed: "+"
- board text removed: "-"
- board text removed: "ESC v1 02/26"
- board text removed: "VBAT"
