File: PCB/ESC_v3/ESC_v3.kicad_pcb (KiCad board)
At the start: 4 copper layers, 42 x 83.5 mm, 144 parts, among them IC1 TLV77333PDBVR, IC2 TCAN3414DR, IC3 DRV8323SRTAR, J1 Conn_01x04_Pin, J10 Conn_01x01_Pin, J3 Conn_01x01_Pin, J4 Conn_01x01_Pin, J5 Conn_01x01_Pin, J6 Conn_01x01_Pin, J7 Conn_01x01_Pin, J8 Conn_01x01_Pin, J9 Conn_01x01_Pin, Q1 NTMFS5C670NLT1G, Q2 NTMFS5C670NLT1G, Q3 NTMFS5C670NLT1G, Q4 NTMFS5C670NLT1G, Q5 NTMFS5C670NLT1G, Q6 NTMFS5C670NLT1G, U3 STM32G474CETx, Y2 24MHz

Commit message: Layout update
Parts:
- removed C26, C51: 100-220uF, Capacitor_SMD:CP_Elec_8x10
- removed C27, C29, C30, C31: 100-220uF, Capacitor_SMD:CP_Elec_6.3x7.7
- added C57: 1600u, SamacSys_Parts:CAPPRD750W80D1600H3200, F.Cu at (155.7, 74.1)
- added C58: 1600u, SamacSys_Parts:CAPPRD750W80D1600H3200, B.Cu at (155.5, 83.6)
- added R50: 100k, Resistor_SMD:R_0603_1608Metric, B.Cu at (129.7, 96.7)
- added R55: 220k, Resistor_SMD:R_0603_1608Metric, B.Cu at (127.9, 99.6)
- added R56: 470k, Resistor_SMD:R_0603_1608Metric, B.Cu at (128.6, 101.1)
- added R57: 1M, Resistor_SMD:R_0603_1608Metric, B.Cu at (127.9, 102.6)
- added S3: CVS-03TB, SamacSys_Parts:CVS03TB, F.Cu at (128.7, 101.1)
- C19: value 100-220uF -> 100n; footprint Capacitor_SMD:CP_Elec_8x10 -> Capacitor_SMD:C_0402_1005Metric
- C32: value 10n -> 100n
- C37: footprint Capacitor_SMD:C_0805_2012Metric -> Capacitor_SMD:C_0603_1608Metric
- moved C19 18.1 mm to (144.2, 84.6)
- moved D7 8.81 mm to (136.1, 99.2), turned to 90 degrees
- moved D10 8.71 mm to (136.1, 102.6), turned to -90 degrees
- moved R33 5.36 mm to (138.6, 99.8)
- moved R49 5.32 mm to (138.6, 102.6)
- moved J10 2.55 mm to (126.2, 92.8)
- moved J8 2.55 mm to (126.2, 90.2)
- moved J9 2.55 mm to (126.2, 95.4)
- moved R54 1.90 mm to (140.9, 94.2)
- moved C32 1.70 mm to (139.1, 94.5), turned to -90 degrees
- moved C37 0.31 mm to (146.8, 78.8)
- moved R44 0.17 mm to (149.6, 79.9)
- moved R45 0.12 mm to (151.1, 79.9)
Connections:
- C19 pad 1: V_BAT -> CAN_ID
- C32 pad 1: Net-(C32-Pad1) -> V_BAT_MEAS
- R52 pad 2: Net-(C32-Pad1) -> Net-(R52-Pad2)
- R53 pad 1: Net-(C32-Pad1) -> Net-(R52-Pad2)
- R54 pad 2: Net-(C32-Pad1) -> Net-(R52-Pad2)
- U3 pad 31: unconnected-(U3-PA9-Pad31) -> CAN_ID
Routing:
- net CAN_ID: track 0.00 -> 34.5 mm, vias 0 -> 2
- net V_BAT: track 64.1 -> 88.3 mm, vias 1 -> 54
- net +3V3: track 97.3 -> 113.4 mm
- net GND: track 54.9 -> 60.8 mm, vias 83 -> 171
- net Net-(C32-Pad1): track 5.01 -> 0.00 mm
- net Net-(S3-COM_1): track 0.00 -> 3.43 mm, vias 0 -> 1
- net Net-(R52-Pad2): track 0.00 -> 3.01 mm
- net Net-(S3-COM_3): track 0.00 -> 2.58 mm, vias 0 -> 1
- net Net-(S3-COM_2): track 0.00 -> 2.08 mm, vias 0 -> 1
- net Net-(D10-A): track 4.14 -> 2.06 mm
- net USART2_RX: track 27.7 -> 25.8 mm
- net V_BAT_MEAS: track 6.79 -> 8.72 mm
- net Net-(D7-A): track 4.14 -> 2.85 mm
- net DBG_LED: track 17.3 -> 16.3 mm
- net USART2_TX: track 16.3 -> 17.2 mm
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Other:
- board text added: "+"
- board text added: "-"
- board text added: "5V"
- board text added: "CAN ID"
- board text added: "CAN_H"
- board text added: "CAN_L"
- board text added: "DBG"
- board text added: "F"
- board text added: "L"
- board text added: "M"
- board text added: "PWR"
- board text added: "R"

Commit message: Layout update
Changed lines of the file:
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@@
 		(at 157.185 45.00775)
 		(size 0.7)
-		(drill 0.4)
+		(drill 0.3)
 		(layers "F.Cu" "B.Cu")
 		(tenting front back)
@@
 		(at 156.335 45.00775)
 		(size 0.7)
-		(drill 0.4)
+		(drill 0.3)
 		(layers "F.Cu" "B.Cu")
 		(tenting front back)
@@
 		(at 154.635 45.00775)
 		(size 0.7)
-		(drill 0.4)
+		(drill 0.3)
 		(layers "F.Cu" "B.Cu")
 		(tenting front back)
@@
 		(at 158.035 45.00775)
 		(size 0.7)
-		(drill 0.4)
+		(drill 0.3)
 		(layers "F.Cu" "B.Cu")
 		(tenting front back)
@@
 		(at 155.485 45.00775)
 		(size 0.7)
-		(drill 0.4)
+		(drill 0.3)
 		(layers "F.Cu" "B.Cu")
 		(tenting front back)
@@
 	)
 	(zone
-		(net 3)
-		(net_name "V_A_PHASE")
-		(layer "F.Cu")
-		(name "$teardrop_padvia$")
-		(hatch none 0.1)
-		(priority 30277)
-		(attr
-			(teardrop
-				(type padvia)
-			)
-		)
-		(connect_pads yes
-			(clearance 0)
-		)
-		(min_thickness 0.0254)
-		(filled_areas_thickness no)
-		(fill yes
-			(thermal_gap 0.5)
-			(thermal_bridge_width 0.5)
-			(island_removal_mode 1)
-			(island_area_min 10)
-		)
-		(polygon
-			(pts
-				(xy 158.152196 44.900064) (xy 158.067367 44.841369) (xy 157.964964 44.815382) (xy 157.85635 44.826315)
-				(xy 157.806513 44.845827) (xy 157.762811 44.874004) (xy 157.729253 44.907722) (xy 157.704456 44.948089)
-				(xy 157.69087 44.990298) (xy 157.687168 45.037314) (xy 157.691725 45.076032) (xy 158.034293 45.007043)
-				(xy 157.691725 45.076032) (xy 157.702226 45.104546) (xy 157.718419 45.118527) (xy 157.759323 45.11773)
-				(xy 157.79492 45.105856) (xy 157.868926 45.086297) (xy 157.905715 45.090474) (xy 157.940064 45.112196)
-			)
-		)
-	)
-	(zone
 		(net 26)
 		(net_name "Net-(D8-A)")
@@
 			)
 		)
+	)
+	(zone
+		(net 3)
+		(net_name "V_A_PHASE")
+		(layer "F.Cu")
+		(name "$teardrop_padvia$")
+		(hatch none 0.1)
+		(priority 30000)
+		(attr
+			(teardrop
+				(type padvia)
+			)
+		)
+		(connect_pads yes
+			(clearance 0)
+		)
+		(min_thickness 0.0254)
+		(filled_areas_thickness no)
+		(fill yes
+			(thermal_gap 0.5)
+			(thermal_bridge_width 0.5)
+			(island_removal_mode 1)
+			(island_area_min 10)
+		)
+		(polygon
+			(pts
+				(xy 158.152196 44.900064) (xy 158.067367 44.841369) (xy 157.964964 44.815382) (xy 157.85635 44.826315)
+				(xy 157.806513 44.845827) (xy 157.762811 44.874004) (xy 157.729253 44.907722) (xy 157.704456 44.948089)
+				(xy 157.69087 44.990298) (xy 157.687168 45.037314) (xy 157.691725 45.076032) (xy 158.034293 45.007043)
+				(xy 157.691725 45.076032) (xy 157.702226 45.104546) (xy 157.718419 45.118527) (xy 157.759323 45.11773)
+				(xy 157.79492 45.105856) (xy 157.868926 45.086297) (xy 157.905715 45.090474) (xy 157.940064 45.112196)
+			)
+		)

Commit message: Update
Parts:
- C32: value 100n -> 10n
- C46, C47, C48: value 100p -> 1000p
- R10, R17, R20, R4, R5, R9: value 4.7Ω -> 10R
- R46, R47, R48: value 33 -> 1k
Connections:
- net TIM17_CH1 renamed TIM8_CH3
- net TIM17_CH1N renamed TIM3_CH4
- net V_BAT renamed +VBAT
- C21 pad 1: +3V3 -> Net-(IC3-DVDD)
- IC3 pad 33: +3V3 -> Net-(IC3-DVDD)
Routing:
- net +3V3: track 113.4 -> 106.8 mm, vias 11 -> 10
- net Net-(IC3-DVDD): track 0.00 -> 3.38 mm, vias 0 -> 1
