File: PCB/ESC_v3/DRVR.kicad_sch (KiCad schematic)
At the start: 18 parts, among them U2 DRV8323SRTAT

Commit message: Layout update
Parts:
- removed R25, R29, R30: 3m, Resistor_SMD:R_2512_6332Metric, symbol Device:R
- removed U2: DRV8323SRTAT, DRV8323SRTAT:QFN50P600X600X80-41N415X415, symbol DRV8323SRTAT:DRV8323SRTAT
- added IC3: DRV8323SRTAR, QFN50P600X600X80-41N-D, symbol SamacSys_Parts:DRV8323SRTAR
- added R25, R29, R30: 1m, RESC6432X110N, symbol SamacSys_Parts:MSMA2512R0010FGM
Connections:
- net +3V3: now also IC3.24 (VREF), IC3.33 (DVDD)
- net CAL: now also IC3.31 (CAL)
- net ENABLE: now also IC3.30 (ENABLE)
- net GND: now also IC3.32 (AGND), IC3.40 (PGND), IC3.41 (EP), R25.1, R29.1, R30.1
- net G_A_H: now also IC3.6 (GHA)
- net G_A_L: now also IC3.8 (GLA)
- net G_B_H: now also IC3.15 (GHB)
- net G_B_L: now also IC3.13 (GLB)
- net G_C_H: now also IC3.16 (GHC)
- net G_C_L: now also IC3.18 (GLC)
- net INHA: now also IC3.34 (INHA)
- net INHB: now also IC3.36 (INHB)
- net INHC: now also IC3.38 (INHC)
- net INLA: now also IC3.35 (INLA)
- net INLB: now also IC3.37 (INLB)
- net INLC: now also IC3.39 (INLC)
- net NFAULT: now also IC3.25 (NFAULT)
- net SCLK: now also IC3.28 (SCLK)
- net SDI: now also IC3.27 (SDI)
- net SDO: now also IC3.26 (SDO)
- net SNA: now also IC3.10 (SNA)
- net SNB: now also IC3.11 (SNB)
- net SNC: now also IC3.20 (SNC)
- net SOA: now also IC3.23 (SOA)
- net SOB: now also IC3.22 (SOB)
- net SOC: now also IC3.21 (SOC)
- net SPA: now also IC3.9 (SPA), R25.2
- net SPB: now also IC3.12 (SPB), R29.2
- net SPC: now also IC3.19 (SPC), R30.2
- net V_A_PHASE: now also IC3.7 (SHA)
- net V_BAT: now also IC3.4 (VM), IC3.5 (VDRAIN)
- net V_B_PHASE: now also IC3.14 (SHB)
- net V_C_PHASE: now also IC3.17 (SHC)
- net nSCS: now also IC3.29 (NSCS)
- net at C20.1: now also IC3.1 (CPL)
- net at C20.2: now also IC3.2 (CPH)
- net at C22.2: now also IC3.3 (VCP)
Other:
- note added: "Driver setup"
- note added: "MSMA2512R0010FGM"
- note added: "according to datasheet"
- note removed: "Driver setup according to datasheet"
- moved on the sheet: C20, C21, C22, C23, C25, C28

Commit message: Layout update
Connections:
- net V_BAT renamed +VBAT
Changed lines of the file:
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@@
 	(wire
 		(pts
+			(xy 118.11 129.54) (xy 118.11 130.81)
+		)
+		(stroke
+			(width 0)
+			(type default)
+		)
+	)
+	(wire
+		(pts
 			(xy 64.77 80.01) (xy 64.77 82.55)
 		)
@@
 	(wire
 		(pts
+			(xy 218.44 83.82) (xy 218.44 85.09)
+		)
+		(stroke
+			(width 0)
+			(type default)
+		)
+	)
+	(wire
+		(pts
 			(xy 130.81 107.95) (xy 134.62 107.95)
 		)
@@
 	(wire
 		(pts
-			(xy 130.81 130.81) (xy 134.62 130.81)
-		)
-		(stroke
-			(width 0)
-			(type default)
-		)
-	)
-	(wire
-		(pts
 			(xy 26.67 80.01) (xy 27.94 80.01)
 		)
@@
 	(wire
 		(pts
+			(xy 118.11 130.81) (xy 134.62 130.81)
+		)
+		(stroke
+			(width 0)
+			(type default)
+		)
+	)
+	(wire
+		(pts
 			(xy 130.81 90.17) (xy 134.62 90.17)
 		)
@@
 		)
 	)
-	(global_label "V_BAT"
-		(shape input)
-		(at 130.81 130.81 180)
-		(fields_autoplaced yes)
-		(effects
-			(font
-				(size 1.27 1.27)
-			)
-			(justify right)
-		)
-		(property "Intersheetrefs" "${INTERSHEET_REFS}"
-			(at 122.4424 130.81 0)
-			(effects
-				(font
-					(size 1.27 1.27)
-				)
-				(justify right)
-				(hide yes)
-			)
-		)
-	)
-	(global_label "V_BAT"
-		(shape input)
-		(at 218.44 85.09 0)
-		(fields_autoplaced yes)
-		(effects
-			(font
-				(size 1.27 1.27)
-			)
-			(justify left)
-		)
-		(property "Intersheetrefs" "${INTERSHEET_REFS}"
-			(at 226.8076 85.09 0)
-			(effects
-				(font
-					(size 1.27 1.27)
-				)
-				(justify left)
-				(hide yes)
-			)
-		)
-	)
 	(global_label "CAL"
 		(shape input)
@@
 	(symbol
 		(lib_id "power:+3V3")
+		(at 218.44 83.82 0)
+		(mirror y)
+		(unit 1)
+		(exclude_from_sim no)
+		(in_bom yes)
+		(on_board yes)
+		(dnp no)
+		(property "Reference" "#PWR059"
+			(at 218.44 87.63 0)
+			(effects
+				(font
+					(size 1.27 1.27)
+				)
+				(hide yes)
+			)
+		)
+		(property "Value" "+VBAT"
+			(at 218.44 80.264 0)
+			(effects
+				(font
+					(size 1.27 1.27)
+				)
+			)
+		)
+		(property "Footprint" ""
+			(at 218.44 83.82 0)
+			(effects
+				(font
+					(size 1.27 1.27)
+				)
+				(hide yes)
+			)
+		)
+		(property "Datasheet" ""
+			(at 218.44 83.82 0)
+			(effects
+				(font
+					(size 1.27 1.27)
+				)
+				(hide yes)
+			)
+		)
+		(property "Description" "Power symbol creates a global label with name \"+3V3\""
+			(at 218.44 83.82 0)
+			(effects
+				(font
+					(size 1.27 1.27)
+				)
+				(hide yes)
+			)
+		)
+		(pin "1"
+		)
+		(instances
+			(project "ESC_v3"
+				(path "/bb7f65bd-c3d2-4eba-8e72-fdc4c3d3399c/c36682af-7334-4ae4-b708-5014138612ef"
+					(reference "#PWR059")
+					(unit 1)
+				)
+			)
+		)
+	)
+	(symbol
+		(lib_id "power:+3V3")
 		(at 86.36 31.75 0)
 		(unit 1)
@@
 					(unit 1)
 				)
+			)
+		)
+	)
+	(symbol
+		(lib_id "power:+3V3")
+		(at 118.11 129.54 0)
+		(mirror y)
+		(unit 1)
+		(exclude_from_sim no)
+		(in_bom yes)
+		(on_board yes)
+		(dnp no)
+		(property "Reference" "#PWR060"
+			(at 118.11 133.35 0)
+			(effects
+				(font
+					(size 1.27 1.27)
+				)
+				(hide yes)
+			)
+		)
+		(property "Value" "+VBAT"
+			(at 118.11 125.984 0)
+			(effects
+				(font
+					(size 1.27 1.27)
+				)
+			)
+		)
+		(property "Footprint" ""
+			(at 118.11 129.54 0)
+			(effects
+				(font
+					(size 1.27 1.27)
+				)
+				(hide yes)
+			)
+		)
+		(property "Datasheet" ""
+			(at 118.11 129.54 0)
+			(effects
+				(font
+					(size 1.27 1.27)
+				)
+				(hide yes)
+			)
+		)
+		(property "Description" "Power symbol creates a global label with name \"+3V3\""
+			(at 118.11 129.54 0)
+			(effects
+				(font
+					(size 1.27 1.27)
+				)
+				(hide yes)
+			)
+		)
+		(pin "1"
+		)
+		(instances
+			(project "ESC_v3"
+				(path "/bb7f65bd-c3d2-4eba-8e72-fdc4c3d3399c/c36682af-7334-4ae4-b708-5014138612ef"
+					(reference "#PWR060")
+					(unit 1)
+				)

Commit message: Update
Connections:
- net +3V3: no longer C21.1, IC3.33 (DVDD)
- new net: C21.1, IC3.33 (DVDD)
Other:
- note added: "220n 50V"
- note added: "22u 25V"
- note added: "2u2 16V"
- note added: "2u2 25V"
- moved on the sheet: C21, C25
