File: PCB/ESC_v3/ESC_v3.kicad_sch (KiCad schematic)
At the start: 80 parts, among them J1 Conn_01x04_Pin, J11 Screw_Terminal_01x01, J2 Screw_Terminal_01x01, Q1 NTMFS2D1N08XT1G, Q2 NTMFS2D1N08XT1G, Q3 NTMFS2D1N08XT1G, Q4 NTMFS2D1N08XT1G, Q5 NTMFS2D1N08XT1G, Q6 NTMFS2D1N08XT1G, U1 SN65HVD232, U4 TCAN334G, U5 TCAN334G, U6 TCAN334G, U7 SN65HVD232

Commit message: Layout update
Parts:
- removed C49: 22n, Capacitor_SMD:C_0805_2012Metric, symbol Device:C
- removed C50: 100n, Capacitor_SMD:C_0805_2012Metric, symbol Device:C
- removed L1: 6.8uH, Inductor_SMD:L_0805_2012Metric_Pad1.05x1.20mm_HandSolder, symbol Device:L
- removed U4: TCAN334G, Package_SO:JEITA_SOIC-8_3.9x4.9mm_P1.27mm, symbol Interface_CAN_LIN:TCAN334G
- removed U5: TCAN334G, Package_SO:SOIC-8_3.9x4.9mm_P1.27mm, symbol Interface_CAN_LIN:TCAN334G
- removed U6: TCAN334G, Package_TO_SOT_SMD:TSOT-23-8, symbol Interface_CAN_LIN:TCAN334G
- removed U7: SN65HVD232, Package_SO:SOIC-8_3.9x4.9mm_P1.27mm, symbol Interface_CAN_LIN:SN65HVD230
- added C1: 1-4u7, Capacitor_SMD:C_0805_2012Metric, symbol Device:C
- added IC1: TLV77333PDBVR, SOT95P280X145-5N, symbol SamacSys_Parts:TLV77333PDBVR
- C44: value 100n -> DNP
- C45: value 22n -> 1u
Connections:
- net +3V3: now also C45.1, IC1.5 (OUT)
- net GND: now also C44.2, C45.2, C1.2, IC1.2 (GND); no longer C44.1, C45.1
- removed net +3V3RAW: C44.2, C45.2, J1.4 (Pin_4)
- new net +5V: C1.1, C44.1, IC1.1 (IN), IC1.3 (EN), J1.4 (Pin_4)

Commit message: Layout update
Parts:
- removed D1: SMCJ28A, Diode_SMD:D_SMC, symbol Diode:1.5SMCxxA
- removed H3: MountingHole_Pad, MountingHole:MountingHole_3.2mm_M3_ISO14580_Pad, symbol Mechanical:MountingHole_Pad
- removed J11, J2: Screw_Terminal_01x01, TerminalBlock_Wuerth:Wuerth_REDCUBE-THR_WP-THRSH_74651173_THR, symbol Connector:Screw_Terminal_01x01
- removed Q1, Q2, Q3, Q4, Q5, Q6: NTMFS2D1N08XT1G, Package_SO:ONSemi_SO-8FL_488AA, symbol Transistor_FET:NTMFS016N06CT1G
- removed U1: SN65HVD232, Package_SO:SOIC-8_3.9x4.9mm_P1.27mm, symbol Interface_CAN_LIN:SN65HVD230
- added C50, C52, C53: 4u7, Capacitor_SMD:C_0805_2012Metric, symbol Device:C
- added D1: SMCJ33A-TR, SMCJ15ATR, symbol SamacSys_Parts:SMCJ33A-TR
- added D10: LED, LED_SMD:LED_0805_2012Metric, symbol Device:LED
- added IC2: TCAN3414DR, SOIC127P600X175-8N, symbol SamacSys_Parts:TCAN3414DR
- added PS1: XT60PW-M, XT60PWM, symbol SamacSys_Parts:XT60PW-M
- added Q1, Q2, Q3, Q4, Q5, Q6: NTMFS5C670NLT1G, NRVTS10100EMFST1G, symbol SamacSys_Parts:NTMFS5C670NLT1G
- added R49: 2k, Resistor_SMD:R_0603_1608Metric, symbol Device:R
- C15, C18, C4: value 1µF/50V -> 4u7
- C16: footprint Capacitor_SMD:C_0805_2012Metric -> Capacitor_SMD:C_0402_1005Metric
Connections:
- net +3V3: now also IC2.3 (VCC), R49.1
- net CAN_H: now also IC2.7 (CANH)
- net CAN_L: now also IC2.6 (CANL)
- net CAN_RX: now also IC2.4 (RXD)
- net CAN_TX: now also IC2.1 (TXD)
- net GND: now also D1.2 (A), D10.1 (K), IC2.2 (GND), IC2.5 (SHDNVIO), IC2.8 (STB), PS1.2 (-)
- net SPA: now also C50.2, Q2.1 (S), Q2.2 (S_2), Q2.3 (S_3)
- net SPB: now also C52.2, Q4.1 (S), Q4.2 (S_2), Q4.3 (S_3)
- net SPC: now also C53.2, Q6.1 (S), Q6.2 (S_2), Q6.3 (S_3)
- net V_A_PHASE: now also Q1.1 (S), Q1.2 (S_2), Q1.3 (S_3), Q2.5 (D), Q2.6 (D), Q2.7 (D), Q2.8 (D), Q2.9 (D)
- net V_BAT: now also C50.1, C52.1, C53.1, D1.1 (K), PS1.1 (+), Q1.5 (D), Q1.6 (D), Q1.7 (D), Q1.8 (D), Q1.9 (D), Q3.5 (D), Q3.6 (D), Q3.7 (D), Q3.8 (D), Q3.9 (D), Q5.5 (D), Q5.6 (D), Q5.7 (D), Q5.8 (D), Q5.9 (D)
- net V_B_PHASE: now also Q3.1 (S), Q3.2 (S_2), Q3.3 (S_3), Q4.5 (D), Q4.6 (D), Q4.7 (D), Q4.8 (D), Q4.9 (D)
- net V_C_PHASE: now also Q5.1 (S), Q5.2 (S_2), Q5.3 (S_3), Q6.5 (D), Q6.6 (D), Q6.7 (D), Q6.8 (D), Q6.9 (D)
- net at C5.2, R11.2, R3.2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: now also Q1.4 (G)
- net at C8.1, R10.2, R14.1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: now also Q4.4 (G)
- net at C7.2, R13.2, R7.2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: now also Q3.4 (G)
- net at C6.1, R12.2, R4.2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: now also Q2.4 (G)
- net at C12.1, R18.2, R20.2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: now also Q6.4 (G)
- net at C11.2, R17.2, R19.2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: now also Q5.4 (G)
- new net: D10.2 (A), R49.2
Other:
- note added: "2u2-4u7/50V"
- note added: "EMZR500ARA221MHA0G"
- moved on the sheet: C16, C17, D9, H4, R51

Commit message: Layout update
Parts:
- removed C19, C26, C51: 100-220uF, Capacitor_SMD:CP_Elec_8x10, symbol Device:C
- removed C27, C29, C30, C31: 100-220uF, Capacitor_SMD:CP_Elec_6.3x7.7, symbol Device:C
- added C57, C58: 1600u, CAPPRD750W80D1600H3200, symbol SamacSys_Parts:ESL108M063AM9AA
Connections:
- net GND: now also C57.2 (-), C58.2 (-)
- net V_BAT renamed +VBAT
- net +VBAT: now also C57.1 (+), C58.1 (+)
Other:
- note added: "4u7/50V"
- note added: "EGPD500ELL162ML30H"
- note removed: "(600-700uF in total)"
- note removed: "2u2-4u7/50V"
- note removed: "50V 3x220uF"
- note removed: "BTM"
- note removed: "C0G/NP0"
- note removed: "DNP Backup if needed later"
- note removed: "EMZR500ARA221MHA0G"
- note removed: "TOP"
- moved on the sheet: C45, D10, R49

Commit message: Layout update
Other:
- note added: "1N4148WS"
Changed lines of the file:
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@@
+		)
+	)
+	(text "1N4148WS"
+		(exclude_from_sim no)
+		(at 148.082 125.222 0)
+		(effects
+			(font
+				(size 1.27 1.27)
+			)
 		)
 	)
@@
 		(exclude_from_sim no)
 		(at 84.074 28.448 0)
+		(effects
+			(font
+				(size 1.27 1.27)
+			)
+		)
+	)
+	(text "1N4148WS"
+		(exclude_from_sim no)
+		(at 215.138 125.984 0)
 		(effects
 			(font
@@
 			)
 		)
+	)
+	(text "1N4148WS"
+		(exclude_from_sim no)
+		(at 78.232 125.222 0)
+		(effects
+			(font
+				(size 1.27 1.27)
+			)
+		)

Commit message: Update
Parts:
- R10, R17, R20, R4, R5, R9: value 4.7Ω -> 10R
