File: PCB/ESC_v3/MCU.kicad_sch (KiCad schematic)
At the start: 44 parts, among them J10 Conn_01x01_Pin, J3 Conn_01x01_Pin, J4 Conn_01x01_Pin, J5 Conn_01x01_Pin, J6 Conn_01x01_Pin, J7 Conn_01x01_Pin, J8 Conn_01x01_Pin, J9 Conn_01x01_Pin, U3 STM32G474CETx, Y2 24MHz

Commit message: Layout update
Connections:
- net +3V3RAW is gone; now on net GND: J4.1 (Pin_1)
- net +3V3: now also J5.1 (Pin_1)
- net GND: no longer J3.1 (Pin_1)
- net SWCLK: now also J6.1 (Pin_1); no longer J5.1 (Pin_1)
- net SWDIO: now also J3.1 (Pin_1); no longer J6.1 (Pin_1)
Changed lines of the file:
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@@
 	)
 	(junction
+		(at 25.4 109.22)
+		(diameter 0)
+		(color 0 0 0 0)
+	)
+	(junction
 		(at 43.18 179.07)
 		(diameter 0)
@@
 	(wire
 		(pts
-			(xy 25.4 109.22) (xy 38.1 109.22)
-		)
-		(stroke
-			(width 0)
-			(type default)
-		)
-	)
-	(wire
-		(pts
 			(xy 35.56 60.96) (xy 35.56 62.23)
 		)
@@
 	(wire
 		(pts
-			(xy 25.4 111.76) (xy 38.1 111.76)
-		)
-		(stroke
-			(width 0)
-			(type default)
-		)
-	)
-	(wire
-		(pts
 			(xy 139.7 67.31) (xy 137.16 67.31)
 		)
@@
 	(wire
 		(pts
+			(xy 26.67 111.76) (xy 25.4 111.76)
+		)
+		(stroke
+			(width 0)
+			(type default)
+		)
+	)
+	(wire
+		(pts
 			(xy 25.4 137.16) (xy 24.13 137.16)
 		)
@@
 	(wire
 		(pts
-			(xy 38.1 107.95) (xy 38.1 109.22)
+			(xy 39.37 113.03) (xy 39.37 114.3)
 		)
 		(stroke
@@
 	(wire
 		(pts
-			(xy 38.1 111.76) (xy 38.1 113.03)
+			(xy 36.83 109.22) (xy 36.83 110.49)
 		)
 		(stroke
@@
 	(wire
 		(pts
+			(xy 24.13 109.22) (xy 25.4 109.22)
+		)
+		(stroke
+			(width 0)
+			(type default)
+		)
+	)
+	(wire
+		(pts
 			(xy 43.18 187.96) (xy 43.18 189.23)
 		)
@@
 	(wire
 		(pts
+			(xy 25.4 109.22) (xy 36.83 109.22)
+		)
+		(stroke
+			(width 0)
+			(type default)
+		)
+	)
+	(wire
+		(pts
 			(xy 35.56 85.09) (xy 36.83 85.09)
 		)
@@
 	(wire
 		(pts
-			(xy 26.67 114.3) (xy 25.4 114.3)
+			(xy 25.4 114.3) (xy 39.37 114.3)
 		)
 		(stroke
@@
 	(global_label "SWDIO"
 		(shape input)
-		(at 26.67 116.84 0)
+		(at 26.67 111.76 0)
 		(fields_autoplaced yes)
 		(effects
@@
 		)
 		(property "Intersheetrefs" "${INTERSHEET_REFS}"
-			(at 35.9974 116.84 0)
+			(at 35.9974 111.76 0)
 			(effects
 				(font
@@
 	(global_label "SWCLK"
 		(shape input)
-		(at 26.67 114.3 0)
+		(at 26.67 116.84 0)
 		(fields_autoplaced yes)
 		(effects
@@
 		)
 		(property "Intersheetrefs" "${INTERSHEET_REFS}"
-			(at 36.3602 114.3 0)
+			(at 36.3602 116.84 0)
 			(effects
 				(font
@@
 	)
 	(symbol
+		(lib_id "power:+3V3")
+		(at 39.37 113.03 0)
+		(mirror y)
+		(unit 1)
+		(exclude_from_sim no)
+		(in_bom yes)
+		(on_board yes)
+		(dnp no)
+		(property "Reference" "#PWR035"
+			(at 39.37 116.84 0)
+			(effects
+				(font
+					(size 1.27 1.27)
+				)
+				(hide yes)
+			)
+		)
+		(property "Value" "+3V3"
+			(at 39.37 109.474 0)
+			(effects
+				(font
+					(size 1.27 1.27)
+				)
+			)
+		)
+		(property "Footprint" ""
+			(at 39.37 113.03 0)
+			(effects
+				(font
+					(size 1.27 1.27)
+				)
+				(hide yes)
+			)
+		)
+		(property "Datasheet" ""
+			(at 39.37 113.03 0)
+			(effects
+				(font
+					(size 1.27 1.27)
+				)
+				(hide yes)
+			)
+		)
+		(property "Description" "Power symbol creates a global label with name \"+3V3\""
+			(at 39.37 113.03 0)
+			(effects
+				(font
+					(size 1.27 1.27)
+				)
+				(hide yes)
+			)
+		)
+		(pin "1"
+		)
+		(instances
+			(project "ESC_v3"
+				(path "/bb7f65bd-c3d2-4eba-8e72-fdc4c3d3399c/cb41d658-ae32-4bca-a5d5-9c7fe787c40c"
+					(reference "#PWR035")
+					(unit 1)
+				)
+			)
+		)
+	)
+	(symbol
 		(lib_id "Device:C")
 		(at 39.37 38.1 180)
@@
 	)
 	(symbol
-		(lib_id "power:+3V3")
-		(at 38.1 107.95 0)
-		(unit 1)
-		(exclude_from_sim no)
-		(in_bom yes)
-		(on_board yes)
-		(dnp no)
-		(property "Reference" "#PWR035"
-			(at 38.1 111.76 0)
-			(effects
-				(font
-					(size 1.27 1.27)
-				)
-				(hide yes)
-			)
-		)
-		(property "Value" "+3V3RAW"
-			(at 37.592 104.394 0)
-			(effects
-				(font
-					(size 1.27 1.27)
-				)
-			)
-		)
-		(property "Footprint" ""
-			(at 38.1 107.95 0)
-			(effects
-				(font
-					(size 1.27 1.27)
-				)
-				(hide yes)
-			)
-		)
-		(property "Datasheet" ""
-			(at 38.1 107.95 0)
-			(effects
-				(font
-					(size 1.27 1.27)
-				)
-				(hide yes)
-			)
-		)
-		(property "Description" "Power symbol creates a global label with name \"+3V3\""
-			(at 38.1 107.95 0)
-			(effects
-				(font
-					(size 1.27 1.27)
-				)
-				(hide yes)
-			)
-		)
-		(pin "1"
-		)
-		(instances
-			(project "ESC_v3"
-				(path "/bb7f65bd-c3d2-4eba-8e72-fdc4c3d3399c/cb41d658-ae32-4bca-a5d5-9c7fe787c40c"
-					(reference "#PWR035")
-					(unit 1)
-				)
-			)
-		)
-	)
-	(symbol
 		(lib_id "Device:C")
 		(at 43.18 57.15 180)
@@
 	(symbol
 		(lib_id "power:GND")
-		(at 38.1 113.03 0)
+		(at 36.83 110.49 0)
 		(unit 1)
 		(exclude_from_sim no)
@@
 		(dnp no)
 		(property "Reference" "#PWR030"
-			(at 38.1 119.38 0)
+			(at 36.83 116.84 0)
 			(effects
 				(font
@@
 		)
 		(property "Value" "GND"
-			(at 38.1 116.586 0)
+			(at 36.83 114.046 0)
 			(effects
 				(font
@@
 		)
 		(property "Footprint" ""
-			(at 38.1 113.03 0)
+			(at 36.83 110.49 0)
 			(effects
 				(font
@@
 		)
 		(property "Datasheet" ""
-			(at 38.1 113.03 0)
+			(at 36.83 110.49 0)
 			(effects
 				(font
@@
 		)
 		(property "Description" "Power symbol creates a global label with name \"GND\" , ground"
-			(at 38.1 113.03 0)
+			(at 36.83 110.49 0)
 			(effects
 				(font

Commit message: Layout update
Parts:
- removed L2: 6.8uH, Inductor_SMD:L_0805_2012Metric_Pad1.05x1.20mm_HandSolder, symbol Device:L
- added C49: 1u, Capacitor_SMD:C_0603_1608Metric, symbol Device:C
- added D7: LED, LED_SMD:LED_0805_2012Metric, symbol Device:LED
- added FB1: FCM1608KF-601T03, Inductor_SMD:L_0603_1608Metric, symbol Device:FerriteBead
- added R32: 10, Resistor_SMD:R_0402_1005Metric, symbol Device:R
- added R33: 2k, Resistor_SMD:R_0603_1608Metric, symbol Device:R
- C35, C43: footprint Capacitor_SMD:C_0603_1608Metric -> Capacitor_SMD:C_0402_1005Metric
- C39, C42: value 1u/DNP -> 1u
- C40, C41: footprint Capacitor_SMD:C_0805_2012Metric -> Capacitor_SMD:C_0603_1608Metric
- C46, C47: value 12pF -> 100p; footprint Capacitor_SMD:C_0603_1608Metric -> Capacitor_SMD:C_0402_1005Metric
- C48: value 12pF -> 100p; footprint Capacitor_SMD:C_0805_2012Metric -> Capacitor_SMD:C_0402_1005Metric
- J10, J3, J4, J5, J6, J7, J8, J9: now not fitted
- R46, R47, R48: value 100 -> 33; footprint Resistor_SMD:R_0603_1608Metric -> Resistor_SMD:R_0402_1005Metric
Connections:
- net +3V3: now also FB1.2
- net +VDDA: now also FB1.1, R32.1; no longer C43.2, U3.20 (VREF+)
- net GND: now also C49.1, D7.1 (K)
- net DBG_LED: now reaches U3.18 (PB2)
- net DBG_LED: now also R33.1
- new net: D7.2 (A), R33.2
- new net +VREF: C43.2, C49.2, R32.2, U3.20 (VREF+)
Other:
- note added: "ABM8W-24.0000MHZ-6-D1X-T3"
- note added: "FCM1608KF-601T03 600 Ω @ 100 MHz, low DC resistance From ST datasheet and BOM"
- note removed: "I think this is what ST recommends"
- note removed: "Maybe: Ferrite bead 600 Ω @ 100 MHz, low DC resistance (Murata BLM18 / BLM21 series)"
- moved on the sheet: C24, C35, C36, C37, C38, C39, C42, C43, R34, R37, R38, R39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

Commit message: Layout update
Parts:
- added C19: 100n, Capacitor_SMD:C_0402_1005Metric, symbol Device:C
- added R50: 100k, Resistor_SMD:R_0603_1608Metric, symbol Device:R
- added R55: 220k, Resistor_SMD:R_0603_1608Metric, symbol Device:R
- added R56: 470k, Resistor_SMD:R_0603_1608Metric, symbol Device:R
- added R57: 1M, Resistor_SMD:R_0603_1608Metric, symbol Device:R
- added S3: CVS-03TB, CVS03TB, symbol SamacSys_Parts:CVS-03TB
- C32: value 10n -> 100n
- C37: footprint Capacitor_SMD:C_0805_2012Metric -> Capacitor_SMD:C_0603_1608Metric
Connections:
- net +3V3: now also R50.2
- net GND: now also C19.2, R55.2, R56.2, R57.2
- net V_BAT_MEAS: now also C32.1
- net at R52.2, R53.1, R54.2: no longer C32.1
- net CAN_ID: now reaches U3.31 (PA9)
- net CAN_ID: now also C19.1, R50.1, S3.B1 (NO_1), S3.B2 (NO_2), S3.B3 (NO_3)
- net V_BAT renamed +VBAT
- new net: R56.1, S3.A2 (COM_2)
- new net: R57.1, S3.A3 (COM_3)
- new net: R55.1, S3.A1 (COM_1)
Other:
- note added: "1: 100k/(470k & 220k) = 1.979 V 2: 100k/(220k & 1M) = 2.123 V 3: 100k/(1M & 470k) = 100k/14.986k = 2.514 V"
- note added: "4: 100k/220k = 2.269 V 5: 100k/470k = 2.721 V 6: 100k/1M = 3 V"
- note added: "CAN device ID setup"
- moved on the sheet: C32, R52, R53, R54, U3

Commit message: Update
Parts:
- C32: value 100n -> 10n
- C46, C47, C48: value 100p -> 1000p
- R46, R47, R48: value 33 -> 1k
Connections:
- net TIM17_CH1 renamed TIM8_CH3
- net TIM17_CH1N renamed TIM3_CH4
Other:
- note added: "Remapped: TIM17_CH1 -> TIM8_CH3 TIM17_CH1N -> TIM3_CH4"
